Commit message: Addedd pseudo inverse of jacobian, and odom of each base are ok

File: src/escalador_description_serial_1/urdf/escalador_serial_1.urdf.xacro (robot description, xacro)
@@ -9,6 +9,6 @@
   <xacro:include filename="$(find escalador_description_serial_1)/urdf/escalador_serial_1_description.urdf.xacro" />
   <xacro:include filename="$(find escalador_description_serial_1)/urdf/escalador_serial_1_control.xacro" />
-  <link name="world"/>
-  <xacro:robot1 parent="world" prefix="$(arg prefix)">
+  <link name="odom1"/>
+  <xacro:robot1 parent="odom1" prefix="$(arg prefix)">
     <origin xyz="0 0 0" rpy="0 0 0" />
   </xacro:robot1>

File: src/escalador_description_serial_1/urdf/escalador_serial_1_description.urdf.xacro (robot description, xacro)
@@ -8,9 +8,9 @@
   </joint>
   <link name="${prefix}end-effector"/>
-  <link name="${prefix}dummy_base"/>
-  <joint name="dummy" type="fixed">
-    <origin rpy="0.0 0.0 0.0" xyz="0.0 0.0 0.0"/>
-    <parent link="${prefix}LINK_7"/>
-    <child link="${prefix}dummy_base"/>
+  <link name="${prefix}end-dummy"/>
+  <joint name="dummy_joint" type="fixed">
+    <origin rpy="0.0 3.14 0.0" xyz="0.0 0.0 0.0"/>
+    <parent link="${prefix}end-effector"/>
+    <child link="${prefix}end-dummy"/>
   </joint>
   <joint name="end_joint" type="fixed">

File: src/escalador_description_serial_2/urdf/escalador_serial_2.urdf.xacro (robot description, xacro)
@@ -9,6 +9,6 @@
   <xacro:include filename="$(find escalador_description_serial_2)/urdf/escalador_serial_2_description.urdf.xacro" />
   <xacro:include filename="$(find escalador_description_serial_2)/urdf/escalador_serial_2_control.xacro" />
-  <link name="world"/>
-  <xacro:robot2 parent="world" prefix="$(arg prefix)">
+  <link name="odom2"/>
+  <xacro:robot2 parent="odom2" prefix="$(arg prefix)">
     <origin xyz="0 0 0" rpy="0 0 0" />
   </xacro:robot2>

File: src/escalador_description_serial_2/urdf/escalador_serial_2_description.urdf.xacro (robot description, xacro)
@@ -8,9 +8,9 @@
   </joint>
   <link name="${prefix}end-effector"/>
-  <link name="${prefix}dummy_base"/>
-  <joint name="dummy" type="fixed">
-    <origin rpy="0.0 0.0 0.0" xyz="0.0 0.0 0.0"/>
-    <parent link="${prefix}LINK_1"/>
-    <child link="${prefix}dummy_base"/>
+  <link name="${prefix}end-dummy"/>
+  <joint name="dummy_joint" type="fixed">
+    <origin rpy="0.0 -3.14 0.0" xyz="0.0 0.0 0.0"/>
+    <parent link="${prefix}end-effector"/>
+    <child link="${prefix}end-dummy"/>
   </joint>
   <joint name="end_joint" type="fixed">

Commit message: Dynamyxel working

File: src/escalador_description_serial_1/urdf/escalador_serial_1.urdf.xacro (robot description, xacro)
@@ -8,10 +8,9 @@
   <xacro:arg name="prefix" default="" />
   <xacro:include filename="$(find escalador_description_serial_1)/urdf/escalador_serial_1_description.urdf.xacro" />
-  <xacro:include filename="$(find escalador_description_serial_1)/urdf/escalador_serial_1_control.xacro" />
+  <xacro:include filename="$(find escalador_description_serial_1)/urdf/escalador_serial_1_ros2_control.xacro" />
   <link name="odom1"/>
   <xacro:robot1 parent="odom1" prefix="$(arg prefix)">
     <origin xyz="0 0 0" rpy="0 0 0" />
   </xacro:robot1>
-  <xacro:robot1_control
-    name="serial_escalador_1" prefix="$(arg prefix)" />
+  <xacro:escalador_serial_1_ros2_control name="escalador_serial_1_ros2_control" />
 </robot>

File: src/escalador_description_serial_1/urdf/escalador_serial_1_description.urdf.xacro (robot description, xacro)
@@ -10,10 +10,10 @@
   <link name="${prefix}end-dummy"/>
   <joint name="dummy_joint" type="fixed">
-    <origin rpy="0.0 3.14 0.0" xyz="0.0 0.0 0.0"/>
+    <origin rpy="0.0 3.14 0.0" xyz="0.0 0.0 0.000"/>
     <parent link="${prefix}end-effector"/>
     <child link="${prefix}end-dummy"/>
   </joint>
   <joint name="end_joint" type="fixed">
-    <origin rpy="0.0 0.0 0.0" xyz="0.0 0.0 0.07100"/>
+    <origin rpy="0.0 0.0 0.0" xyz="0.0 0.0 0.07400"/>
     <parent link="${prefix}LINK_7"/>
     <child link="${prefix}end-effector"/>

File: src/escalador_description_serial_2/urdf/escalador_serial_2.urdf.xacro (robot description, xacro)
@@ -8,10 +8,9 @@
   <xacro:arg name="prefix" default="" />
   <xacro:include filename="$(find escalador_description_serial_2)/urdf/escalador_serial_2_description.urdf.xacro" />
-  <xacro:include filename="$(find escalador_description_serial_2)/urdf/escalador_serial_2_control.xacro" />
+  <xacro:include filename="$(find escalador_description_serial_2)/urdf/escalador_serial_2_ros2_control.xacro" />
   <link name="odom2"/>
   <xacro:robot2 parent="odom2" prefix="$(arg prefix)">
     <origin xyz="0 0 0" rpy="0 0 0" />
   </xacro:robot2>
-  <xacro:robot2_control
-    name="serial_escalador_2" prefix="$(arg prefix)" />
+  <xacro:robot2_ros2_control name ="robot2ctr" prefix="$(arg prefix)" />
 </robot>

File: src/escalador_description_serial_2/urdf/escalador_serial_2_description.urdf.xacro (robot description, xacro)
@@ -10,10 +10,10 @@
   <link name="${prefix}end-dummy"/>
   <joint name="dummy_joint" type="fixed">
-    <origin rpy="0.0 -3.14 0.0" xyz="0.0 0.0 0.0"/>
+    <origin rpy="0.0 -3.14 0.0" xyz="0.0 0.0 0.000"/>
     <parent link="${prefix}end-effector"/>
     <child link="${prefix}end-dummy"/>
   </joint>
   <joint name="end_joint" type="fixed">
-    <origin rpy="0.0 0.0 0.0" xyz="0.0 0.0 0.07100"/>
+    <origin rpy="0.0 0.0 0.0" xyz="0.0 0.0 0.06900"/>
     <parent link="${prefix}LINK_1"/>
     <child link="${prefix}end-effector"/>
