Commit message: add joints logic to each base

File: src/escalador_description_serial_1/urdf/escalador_serial_1_description.urdf.xacro (robot description, xacro)
@@ -2,8 +2,14 @@
 <robot xmlns:xacro="http://www.ros.org/wiki/xacro">
   <xacro:macro name="robot1" params="parent prefix *origin">
-    <joint name="${prefix}base_joint" type="fixed">
+  <joint name="${prefix}base_joint" type="fixed">
     <xacro:insert_block name="origin" />
     <parent link="${parent}"/>
     <child link="${prefix}LINK_1" />
+  </joint>
+  <link name="${prefix}end-effector"/>
+  <joint name="end_joint" type="fixed">
+    <origin rpy="0.0 0.0 0.0" xyz="0.0 0.0 0.07100"/>
+    <parent link="${prefix}LINK_7"/>
+    <child link="${prefix}end-effector"/>
   </joint>
   <joint name="J1" type="revolute">

File: src/escalador_description_serial_2/urdf/escalador_serial_2_description.urdf.xacro (robot description, xacro)
@@ -6,4 +6,10 @@
     <parent link="${parent}"/>
     <child link="${prefix}LINK_7" />
+  </joint>
+  <link name="${prefix}end-effector"/>
+  <joint name="end_joint" type="fixed">
+    <origin rpy="0.0 0.0 0.0" xyz="0.0 0.0 0.07100"/>
+    <parent link="${prefix}LINK_1"/>
+    <child link="${prefix}end-effector"/>
   </joint>
  <joint name="J1" type="revolute">

Commit message: base changes fixed

File: src/escalador_description_serial_1/urdf/escalador_serial_1_description.urdf.xacro (robot description, xacro)
@@ -8,4 +8,10 @@
   </joint>
   <link name="${prefix}end-effector"/>
+  <link name="${prefix}dummy_base"/>
+  <joint name="dummy" type="fixed">
+    <origin rpy="0.0 0.0 0.0" xyz="0.0 0.0 0.07100"/>
+    <parent link="${prefix}LINK_7"/>
+    <child link="${prefix}dummy_base"/>
+  </joint>
   <joint name="end_joint" type="fixed">
     <origin rpy="0.0 0.0 0.0" xyz="0.0 0.0 0.07100"/>

File: src/escalador_description_serial_2/urdf/escalador_serial_2_description.urdf.xacro (robot description, xacro)
@@ -8,4 +8,10 @@
   </joint>
   <link name="${prefix}end-effector"/>
+  <link name="${prefix}dummy_base"/>
+  <joint name="dummy" type="fixed">
+    <origin rpy="0.0 0.0 0.0" xyz="0.0 0.0 0.07100"/>
+    <parent link="${prefix}LINK_1"/>
+    <child link="${prefix}dummy_base"/>
+  </joint>
   <joint name="end_joint" type="fixed">
     <origin rpy="0.0 0.0 0.0" xyz="0.0 0.0 0.07100"/>

Commit message: odometry added

File: src/escalador_description_serial_1/urdf/escalador_serial_1_description.urdf.xacro (robot description, xacro)
@@ -10,5 +10,5 @@
   <link name="${prefix}dummy_base"/>
   <joint name="dummy" type="fixed">
-    <origin rpy="0.0 0.0 0.0" xyz="0.0 0.0 0.07100"/>
+    <origin rpy="0.0 0.0 0.0" xyz="0.0 0.0 0.0"/>
     <parent link="${prefix}LINK_7"/>
     <child link="${prefix}dummy_base"/>

File: src/escalador_description_serial_2/urdf/escalador_serial_2_description.urdf.xacro (robot description, xacro)
@@ -10,5 +10,5 @@
   <link name="${prefix}dummy_base"/>
   <joint name="dummy" type="fixed">
-    <origin rpy="0.0 0.0 0.0" xyz="0.0 0.0 0.07100"/>
+    <origin rpy="0.0 0.0 0.0" xyz="0.0 0.0 0.0"/>
     <parent link="${prefix}LINK_1"/>
     <child link="${prefix}dummy_base"/>

Commit message: last working version

File: src/escalador_description_serial_1/urdf/escalador_serial_1_description.urdf.xacro (robot description, xacro)
@@ -10,4 +10,5 @@
   <link name="${prefix}end-dummy"/>
   <joint name="dummy_joint" type="fixed">
+    <limit upper="0" lower="0" effort="0" velocity="0"/>
     <origin rpy="0.0 3.14 0.0" xyz="0.0 0.0 0.000"/>
     <parent link="${prefix}end-effector"/>
@@ -15,10 +16,11 @@
   </joint>
   <joint name="end_joint" type="fixed">
-    <origin rpy="0.0 0.0 0.0" xyz="0.0 0.0 0.07400"/>
+    <limit upper="0" lower="0" effort="0" velocity="0"/>
+    <origin rpy="0.0 0.0 0.0" xyz="0.0 0.0 0.07100"/>
     <parent link="${prefix}LINK_7"/>
     <child link="${prefix}end-effector"/>
   </joint>
   <joint name="J1" type="revolute">
-    <limit lower="-3.14000" upper="3.14000" effort="0.00000" velocity="0.00000"/>
+    <limit lower="-6.28000" upper="6.28000" effort="0.00000" velocity="0.00000"/>
     <origin rpy="-0.00000 -0.00000 3.14159" xyz="0.00000 -0.00000 0.07100"/>
     <parent link="${prefix}LINK_1"/>
@@ -41,5 +43,5 @@
   </joint>
   <joint name="J4" type="revolute">
-    <limit lower="-3.14000" upper="3.14000" effort="0.00000" velocity="0.00000"/>
+    <limit lower="-6.28000" upper="6.28000" effort="0.00000" velocity="0.00000"/>
     <origin rpy="1.57080 0.00000 0.00000" xyz="-0.00000 -0.13800 -0.00000"/>
     <parent link="${prefix}LINK_4"/>
@@ -55,5 +57,5 @@
   </joint>
   <joint name="J6" type="revolute">
-    <limit lower="-3.14000" upper="3.14000" effort="0.00000" velocity="0.00000"/>
+    <limit lower="-6.28000" upper="6.28000" effort="0.00000" velocity="0.00000"/>
     <origin rpy="1.57080 0.00000 0.00000" xyz="-0.00000 -0.10900 -0.00000"/>
     <parent link="${prefix}LINK_6"/>
@@ -69,7 +71,9 @@
     </collision>
     <inertial>
-      <inertia ixx="0.00048" ixy="0.00000" ixz="0.00006" iyy="0.00077" iyz="0.00000" izz="0.00059"/>
-      <origin rpy="0.00000 0.00000 0.00000" xyz="0.00889 0.00002 0.02822"/>
-      <mass value="1.50000"/>
+      <origin xyz="-0.011218 -0.000000 0.018785" rpy="0 0 0"/>
+      <mass value="0.375"/>
+      <inertia ixx="0.000108994"
+              ixy="-0.000000000" iyy="0.000198249"
+              ixz="0.000016726" iyz="-0.000000000" izz="0.000200988" />
     </inertial>
     <visual name="LINK_1_visual">
@@ -77,5 +81,5 @@
       <material name="SILVER"/>
       <geometry>
-        <mesh filename="file://$(find escalador_description_serial_1)/meshes/ON-OFF-PAW-Alumínio_MEF.148.dae" scale="0.00100 0.00100 0.00100"/>
+        <mesh filename="file://$(find escalador_description_serial_1)/meshes/pata_1.dae" scale="0.00100 0.00100 0.00100"/>
       </geometry>
     </visual>
@@ -89,7 +93,9 @@
     </collision>
     <inertial>
-      <inertia ixx="0.00088" ixy="-0.00000" ixz="-0.00000" iyy="0.00071" iyz="-0.00009" izz="0.00031"/>
-      <origin rpy="0.00000 0.00000 0.00000" xyz="-0.00000 0.00420 0.05390"/>
-      <mass value="1.50000"/>
+      <origin xyz="-0.000005 -0.008676 0.052092" rpy="0 0 0"/>
+      <mass value="0.354"/>
+      <inertia ixx="0.000223854"
+              ixy="0.000000016" iyy="0.000146294"
+              ixz="-0.000000107" iyz="-0.000034608" izz="0.000151022" />
     </inertial>
     <visual name="LINK_2_visual">
@@ -109,7 +115,9 @@
     </collision>
     <inertial>
-      <inertia ixx="0.00640" ixy="0.00000" ixz="0.00001" iyy="0.00638" iyz="-0.00009" izz="0.00033"/>
-      <origin rpy="0.00000 0.00000 0.00000" xyz="-0.00001 -0.10623 0.00117"/>
-      <mass value="1.50000"/>
+      <origin xyz="-0.000017 -0.000742 0.101033" rpy="0 0 0"/>
+      <mass value="0.477"/>
+      <inertia ixx="0.002864655"
+                ixy="-0.000000004" iyy="0.002867671"
+                ixz="0.000000689" iyz="-0.000000419" izz="0.000140001" />
     </inertial>
     <visual name="LINK_3_visual">
@@ -129,7 +137,9 @@
     </collision>
     <inertial>
-      <inertia ixx="0.00063" ixy="-0.00000" ixz="0.00000" iyy="0.00054" iyz="0.00007" izz="0.00014"/>
-      <origin rpy="0.00000 0.00000 0.00000" xyz="-0.00009 -0.07515 -0.00263"/>
-      <mass value="1.50000"/>
+        <origin xyz="0.000000 -0.009079 0.081987" rpy="0 0 0"/>
+        <mass value="0.372"/>
+        <inertia ixx="0.000135253"
+                ixy="-0.000000000" iyy="0.000047636"
+                ixz="-0.000000000" iyz="0.000000471" izz="0.000162513" />
     </inertial>
     <visual name="LINK_4_visual">
@@ -149,8 +159,10 @@
     </collision>
     <inertial>
-      <inertia ixx="0.00064" ixy="-0.00000" ixz="0.00000" iyy="0.00056" iyz="0.00001" izz="0.00027"/>
-      <origin rpy="0.00000 0.00000 0.00000" xyz="-0.00007 0.00099 0.03555"/>
-      <mass value="1.50000"/>
-    </inertial>
+        <origin xyz="0.000000 -0.001015 -0.021991" rpy="0 0 0"/>
+        <mass value="0.202"/>
+        <inertia ixx="0.000117912"
+                ixy="-0.000000000" iyy="0.000105186"
+                ixz="-0.000000000" iyz="0.000003166" izz="0.000048390" />
+      </inertial>
     <visual name="LINK_5_visual">
       <origin rpy="-1.57080 -0.52299 0.00000" xyz="0.00000 -0.00000 -0.00000"/>
@@ -169,7 +181,9 @@
     </collision>
     <inertial>
-      <inertia ixx="0.00454" ixy="0.00000" ixz="-0.00000" iyy="0.00364" iyz="0.00044" izz="0.00158"/>
-      <origin rpy="0.00000 0.00000 0.00000" xyz="-0.00000 -0.05424 -0.00420"/>
-      <mass value="1.50000"/>
+        <origin xyz="-0.000005 -0.008676 0.052092" rpy="0 0 0"/>
+        <mass value="0.354"/>
+        <inertia ixx="0.000223854"
+                ixy="0.000000016" iyy="0.000146294"
+                ixz="-0.000000107" iyz="-0.000034608" izz="0.000151022" />
     </inertial>
     <visual name="LINK_6_visual">
@@ -189,7 +203,9 @@
     </collision>
     <inertial>
-      <inertia ixx="0.00049" ixy="-0.00000" ixz="0.00006" iyy="0.00079" iyz="-0.00000" izz="0.00061"/>
-      <origin rpy="0.00000 0.00000 0.00000" xyz="-0.00889 0.00002 0.04190"/>
-      <mass value="1.50000"/>
+        <origin xyz="-0.011218 -0.000000 0.018785" rpy="0 0 0"/>
+        <mass value="0.375"/>
+        <inertia ixx="0.000108994"
+                ixy="-0.000000000" iyy="0.000198249"
+                ixz="0.000016726" iyz="-0.000000000" izz="0.000200988" />
     </inertial>
     <visual name="LINK_7_visual">
@@ -197,5 +213,5 @@
       <material name="ROBO"/>
       <geometry>
-        <mesh filename="file://$(find escalador_description_serial_1)/meshes/ON-OFF-PAW-Alumínio_MEF.050.dae" scale="0.00100 0.00100 0.00100"/>
+        <mesh filename="file://$(find escalador_description_serial_1)/meshes/pata_2.dae" scale="0.00100 0.00100 0.00100"/>
       </geometry>
     </visual>

File: src/escalador_description_serial_1/urdf/escalador_serial_1_ros2_control.xacro (robot description, xacro)
@@ -11,4 +11,7 @@
       <joint name="J1">
         <param name="id">1</param>
+        <param name="Position_P_Gain">15000</param>
+        <param name="Position_I_Gain">200</param>
+        <param name="Position_D_Gain">100</param>
         <command_interface name="position"/>
         <command_interface name="velocity"/>
@@ -19,4 +22,7 @@
       <joint name="J2">
         <param name="id">2</param>
+        <param name="Position_P_Gain">15000</param>
+        <param name="Position_I_Gain">200</param>
+        <param name="Position_D_Gain">100</param>
         <command_interface name="position"/>
         <command_interface name="velocity"/>
@@ -27,4 +33,7 @@
       <joint name="J3">
         <param name="id">3</param>
+        <param name="Position_P_Gain">15000</param>
+        <param name="Position_I_Gain">200</param>
+        <param name="Position_D_Gain">100</param>
         <command_interface name="position"/>
         <command_interface name="velocity"/>
@@ -35,4 +44,7 @@
       <joint name="J4">
         <param name="id">4</param>
+        <param name="Position_P_Gain">15000</param>
+        <param name="Position_I_Gain">200</param>
+        <param name="Position_D_Gain">100</param>
         <command_interface name="position"/>
         <command_interface name="velocity"/>
@@ -43,4 +55,7 @@
       <joint name="J5">
         <param name="id">5</param>
+        <param name="Position_P_Gain">15000</param>
+        <param name="Position_I_Gain">200</param>
+        <param name="Position_D_Gain">100</param>
         <command_interface name="position"/>
         <command_interface name="velocity"/>
@@ -51,4 +66,7 @@
       <joint name="J6">
         <param name="id">6</param>
+        <param name="Position_P_Gain">15000</param>
+        <param name="Position_I_Gain">200</param>
+        <param name="Position_D_Gain">100</param>
         <command_interface name="position"/>
         <command_interface name="velocity"/>
@@ -58,5 +76,8 @@
       </joint>
       <joint name="BASE1">
-        <param name="id">10</param>
+        <param name="id">20</param>
+        <param name="Position_P_Gain">15000</param>
+        <param name="Position_I_Gain">200</param>
+        <param name="Position_D_Gain">100</param>
         <command_interface name="position"/>
         <command_interface name="velocity"/>
@@ -66,5 +87,8 @@
       </joint>
       <joint name="BASE2">
-        <param name="id">20</param>
+        <param name="id">10</param>
+        <param name="Position_P_Gain">15000</param>
+        <param name="Position_I_Gain">200</param>
+        <param name="Position_D_Gain">100</param>
         <command_interface name="position"/>
         <command_interface name="velocity"/>

File: src/escalador_description_serial_2/urdf/escalador_serial_2_description.urdf.xacro (robot description, xacro)
@@ -15,10 +15,10 @@
   </joint>
   <joint name="end_joint" type="fixed">
-    <origin rpy="0.0 0.0 0.0" xyz="0.0 0.0 0.06900"/>
+    <origin rpy="0.0 0.0 0.0" xyz="0.0 0.0 0.07100"/>
     <parent link="${prefix}LINK_1"/>
     <child link="${prefix}end-effector"/>
   </joint>
  <joint name="J1" type="revolute">
-    <limit lower="-3.14000" upper="3.14000" effort="0.00000" velocity="0.00000"/>
+    <limit lower="-6.28000" upper="6.28000" effort="0.00000" velocity="0.00000"/>
     <origin rpy="1.57080 -0.00000 0.00000" xyz="0.00000 -0.10900 0.00000"/>
     <parent link="${prefix}LINK_2"/>
@@ -34,5 +34,5 @@
   </joint>
   <joint name="J3" type="revolute">
-    <limit lower="-3.14000" upper="3.14000" effort="0.00000" velocity="0.00000"/>
+    <limit lower="-6.28000" upper="6.28000" effort="0.00000" velocity="0.00000"/>
     <origin rpy="-3.00824 1.57080 1.70415" xyz="-0.00000 -0.00000 0.13800"/>
     <parent link="${prefix}LINK_4"/>
@@ -55,5 +55,5 @@
   </joint>
   <joint name="J6" type="revolute">
-    <limit lower="-3.14000" upper="3.14000" effort="0.00000" velocity="0.00000"/>
+    <limit lower="-6.28000" upper="6.28000" effort="0.00000" velocity="0.00000"/>
     <origin rpy="-0.00000 0.00000 -3.14159" xyz="-0.00000 -0.00000 0.07100"/>
     <parent link="${prefix}LINK_7"/>
@@ -71,5 +71,5 @@
       <inertia ixx="0.00065" ixy="0.00000" ixz="0.00008" iyy="0.00105" iyz="0.00000" izz="0.00081"/>
       <origin rpy="0.00000 0.00000 0.00000" xyz="-0.00889 0.00002 0.04189"/>
-      <mass value="1.50000"/>
+      <mass value="0.47000"/>
     </inertial>
     <visual name="LINK_1_visual">
@@ -77,5 +77,5 @@
       <material name="SILVER"/>
       <geometry>
-        <mesh filename="file://$(find escalador_description_serial_2)/meshes/ON-OFF-PAW-Alumínio_MEF.148.dae" scale="0.00100 0.00100 0.00100"/>
+        <mesh filename="file://$(find escalador_description_serial_2)/meshes/pata_1.dae" scale="0.00100 0.00100 0.00100"/>
       </geometry>
     </visual>
@@ -91,5 +91,5 @@
       <inertia ixx="0.00163" ixy="0.00000" ixz="0.00000" iyy="0.00131" iyz="-0.00016" izz="0.00057"/>
       <origin rpy="0.00000 0.00000 0.00000" xyz="-0.00000 -0.05421 -0.00420"/>
-      <mass value="1.50000"/>
+      <mass value="0.47000"/>
     </inertial>
     <visual name="LINK_2_visual">
@@ -111,5 +111,5 @@
       <inertia ixx="0.00675" ixy="0.00000" ixz="-0.00001" iyy="0.00674" iyz="0.00009" izz="0.00034"/>
       <origin rpy="0.00000 0.00000 0.00000" xyz="-0.09288 -0.00001 0.00117"/>
-      <mass value="1.50000"/>
+      <mass value="0.47000"/>
     </inertial>
     <visual name="LINK_3_visual">
@@ -131,5 +131,5 @@
       <inertia ixx="0.00250" ixy="0.00000" ixz="-0.00000" iyy="0.00216" iyz="0.00028" izz="0.00058"/>
       <origin rpy="0.00000 0.00000 0.00000" xyz="-0.00009 0.00263 0.06197"/>
-      <mass value="1.50000"/>
+      <mass value="0.47000"/>
     </inertial>
     <visual name="LINK_4_visual">
@@ -151,5 +151,5 @@
       <inertia ixx="0.00083" ixy="0.00000" ixz="-0.00000" iyy="0.00073" iyz="0.00001" izz="0.00035"/>
       <origin rpy="0.00000 0.00000 0.00000" xyz="-0.00007 0.02556 0.00099"/>
-      <mass value="1.50000"/>
+      <mass value="0.47000"/>
     </inertial>
     <visual name="LINK_5_visual">
@@ -171,5 +171,5 @@
       <inertia ixx="0.00164" ixy="-0.00000" ixz="0.00000" iyy="0.00131" iyz="0.00016" izz="0.00057"/>
       <origin rpy="0.00000 0.00000 0.00000" xyz="-0.00000 0.00420 0.05387"/>
-      <mass value="1.50000"/>
+      <mass value="0.47000"/>
     </inertial>
     <visual name="LINK_6_visual">
@@ -191,5 +191,5 @@
       <inertia ixx="0.00065" ixy="-0.00000" ixz="0.00008" iyy="0.00105" iyz="-0.00000" izz="0.00081"/>
       <origin rpy="0.00000 0.00000 0.00000" xyz="0.00889 0.00002 0.02822"/>
-      <mass value="1.50000"/>
+      <mass value="0.47000"/>
     </inertial>
     <visual name="LINK_7_visual">
@@ -197,5 +197,5 @@
       <material name="ROBO"/>
       <geometry>
-        <mesh filename="file://$(find escalador_description_serial_2)/meshes/ON-OFF-PAW-Alumínio_MEF.050.dae" scale="0.00100 0.00100 0.00100"/>
+        <mesh filename="file://$(find escalador_description_serial_2)/meshes/pata_2.dae" scale="0.00100 0.00100 0.00100"/>
       </geometry>
     </visual>

File: src/escalador_description_serial_2/urdf/escalador_serial_2_ros2_control.xacro (robot description, xacro)
@@ -5,10 +5,12 @@
       <hardware>
         <plugin>dynamixel_hardware/DynamixelHardware</plugin>
-        <param name="usb_port">/dev/ttyUSB0</param>
-        <param name="baud_rate">1000000</param>
-        <!-- <param name="use_dummy">true</param> -->
+         <param name="usb_port">/dev/ttyUSB0</param>
+         <param name="baud_rate">1000000</param>
+         <param name="use_dummy">true</param>
       </hardware>
       <joint name="J1">
         <param name="id">01</param>
+        <param name="offset">3.14</param>
+        <param name="Profile_Velocity">20</param>
         <command_interface name="position"/>
         <command_interface name="velocity"/>
@@ -19,4 +21,6 @@
       <joint name="J2">
         <param name="id">02</param>
+        <param name="offset">3.12</param>
+        <param name="Profile_Velocity">20</param>
         <command_interface name="position"/>
         <command_interface name="velocity"/>
@@ -27,4 +31,6 @@
       <joint name="J3">
         <param name="id">03</param>
+        <param name="offset">3.17</param>
+        <param name="Profile_Velocity">20</param>
         <command_interface name="position"/>
         <command_interface name="velocity"/>
@@ -35,4 +41,6 @@
       <joint name="J4">
         <param name="id">04</param>
+        <param name="offset">3.14</param>
+        <param name="Profile_Velocity">20</param>
         <command_interface name="position"/>
         <command_interface name="velocity"/>
@@ -43,4 +51,6 @@
       <joint name="J5">
         <param name="id">05</param>
+        <param name="offset">3.14</param>
+        <param name="Profile_Velocity">20</param>
         <command_interface name="position"/>
         <command_interface name="velocity"/>
@@ -51,4 +61,6 @@
       <joint name="J6">
         <param name="id">06</param>
+        <param name="offset">3.14</param>
+        <param name="Profile_Velocity">20</param>
         <command_interface name="position"/>
         <command_interface name="velocity"/>
@@ -58,5 +70,6 @@
       </joint>
       <joint name ="BASE1">
-        <param name="id">20</param>
+        <param name="offset">1.57</param>
+        <param name="id">10</param>
         <command_interface name="position"/>
         <command_interface name="velocity"/>
@@ -66,5 +79,6 @@
       </joint>
       <joint name ="BASE2">
-        <param name="id">10</param>
+        <param name="offset">1.57</param>
+        <param name="id">20</param>
         <command_interface name="position"/>
         <command_interface name="velocity"/>
